File: ThumbsUp.sch (KiCad schematic (older format))
At the start: 159 parts, among them J19 52559-1233, J32 Battery, SW2 SW_DIP_x01, U1 nice_nano

Commit message: Replaced the diodes to the tiny D523 ones, started the tracks.
Parts:
- D1, D10, D11, D12, D13, D14, D15, D16, D17, D18, D19, D2, D20, D21, D22, D23, D24, D25, D26, D27, D28, D29, D3, D30, D31, D32, D33, D34, D35, D36, D37, D38, D39, D4, D40, D41, D42, D43, D44, D45, D46, D47, D48, D49, D5, D50, D51, D52, D53, D54, D55, D56, D57, D58, D6, D7, D8, D9: footprint Diode_SMD:D_SOD-123 -> Diode_SMD:D_SOD-523
