File: ThumbsUp.kicad_pcb (KiCad board)
At the start: 2 copper layers, 282 x 464.4 mm, 163 parts, among them J19 52559-1233, J32 Battery, SW2 SW_DIP_x01, U1 ProMicro

Commit message: Updated the schematics, replaced the switches with MX/Kailh Choc combo
Parts:
- removed G*** (x4): LOGO, Silkscreens:Crowfeet
- MX1, MX10, MX11, MX12, MX13, MX14, MX15, MX16, MX17, MX18, MX19, MX2, MX20, MX21, MX22, MX23, MX24, MX25, MX26, MX27, MX28, MX29, MX3, MX30, MX31, MX32, MX33, MX34, MX35, MX36, MX37, MX38, MX39, MX4, MX40, MX41, MX42, MX43, MX44, MX45, MX46, MX47, MX48, MX49, MX5, MX50, MX51, MX52, MX53, MX54, MX55, MX56, MX57, MX58, MX6, MX7, MX8, MX9: footprint keyswitches:PG1350_GLv2 -> keyswitches:PG1350_MX_sockets
- U1: value ProMicro -> nice_nano; footprint promicro:ProMicro -> nice-nano-kicad:nice_nano
- moved U1 0.17 mm to (143.5, 83.3)
- turned MX31 to 202 degrees
- turned MX32 to 202 degrees
- turned MX33 to 202 degrees
- turned MX34 to 202 degrees
- turned MX35 to 202 degrees
- turned MX36 to 202 degrees
- turned MX37 to 202 degrees
- turned MX38 to 202 degrees
- turned MX39 to 202 degrees
- turned MX40 to 202 degrees
- turned MX41 to 202 degrees
- turned MX42 to 202 degrees
- turned MX43 to 202 degrees
- turned MX44 to 202 degrees
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Connections:
- J19 pad 4: (no net) -> DR-TOP
- JF13 pad 4: GND -> DR
- JM13 pad 4: L3GND -> DR-TOP
Routing:
- net DR: track 0.00 -> 11.4 mm
- net COL1: track 193.7 -> 202.4 mm
- net ROWL2: track 62.2 -> 55.1 mm
- net GND: track 391.5 -> 398.0 mm
- net Net-(JF23-Pad2): track 115.3 -> 110.1 mm
- net SCL: track 95.9 -> 101.0 mm
- net COL0: track 153.6 -> 157.4 mm, vias 2 -> 3
- net SDA: track 97.1 -> 100.5 mm
- net COL4: track 401.6 -> 398.7 mm
- net Net-(JF23-Pad1): track 132.7 -> 129.9 mm
- net COL3: track 359.3 -> 361.3 mm, vias 5 -> 4
- net COL5: track 400.1 -> 401.8 mm
- net COL2: track 397.0 -> 398.8 mm, vias 3 -> 2
- net ROWL1: track 49.6 -> 48.7 mm
- net ROWL4: track 110.7 -> 111.4 mm
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Other:
- outline, holes or cut-outs redrawn
- board text added: "ThumbsUp! v11 ProMicro/nice!nano v2 Kailh Choc and MX Hot-Swap Sockets u/ak66666, May 24, 2025"
- board text removed: "ThumbsUp! v8 ProMicro Kailh Choc/Gat Low Profile Hot-Swap Sockets u/ak66666, Oct 01, 2023"

Commit message: Replaced the diodes to the tiny D523 ones, started the tracks.
Parts:
- D1, D10, D11, D12, D13, D14, D15, D16, D17, D18, D19, D2, D20, D21, D22, D23, D24, D25, D26, D27, D28, D29, D3, D30, D31, D32, D33, D34, D35, D36, D37, D38, D39, D4, D40, D41, D42, D43, D44, D45, D46, D47, D48, D49, D5, D50, D51, D52, D53, D54, D55, D56, D57, D58, D6, D7, D8, D9: footprint Diode_SMD:D_SOD-123 -> Diode_SMD:D_SOD-523
- moved D38 39.5 mm to (164.6, 80.0), turned to 0 degrees
- moved D37 38.4 mm to (164.6, 81.5), turned to 0 degrees
- moved D26 38.1 mm to (158.5, 81.3)
- moved D36 37.5 mm to (164.6, 83.0), turned to 0 degrees
- moved D35 36.9 mm to (164.6, 84.4), turned to 0 degrees
- moved D31 36.0 mm to (158.5, 78.3)
- moved D55 35.9 mm to (156.3, 66.0)
- moved D54 35.4 mm to (156.3, 69.0)
- moved D27 35.0 mm to (164.5, 87.5)
- moved D32 35.0 mm to (158.5, 76.9)
- moved D56 35.0 mm to (156.3, 64.6)
- moved D57 34.0 mm to (156.3, 63.1)
- moved D33 34.0 mm to (158.5, 75.4)
- moved D58 33.1 mm to (156.3, 61.7)
- moved D34 32.9 mm to (158.5, 74.0)
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Routing:
- net COL5: track 401.8 -> 115.9 mm, vias 11 -> 1
- net COL4: track 398.7 -> 141.3 mm, vias 4 -> 1
- net COL2: track 398.8 -> 191.7 mm, vias 2 -> 1
- net Net-(JF33-Pad4): track 214.2 -> 16.5 mm, vias 1 -> 0
- net GND: track 398.0 -> 206.8 mm
- net COL3: track 361.3 -> 177.1 mm, vias 4 -> 1
- net Net-(JF20-Pad1): track 179.1 -> 0.00 mm, vias 1 -> 0
- net Net-(JF33-Pad3): track 191.4 -> 16.4 mm, vias 1 -> 0
- net Net-(JF20-Pad2): track 160.2 -> 0.00 mm, vias 1 -> 0
- net Net-(JF33-Pad2): track 169.4 -> 16.3 mm, vias 1 -> 0
- net Net-(JF33-Pad1): track 150.6 -> 16.1 mm, vias 1 -> 0
- net Net-(JF20-Pad3): track 133.4 -> 0.00 mm, vias 1 -> 0
- net Net-(JF23-Pad1): track 129.9 -> 6.39 mm, vias 1 -> 0
- net Net-(JF28-Pad1): track 122.7 -> 0.00 mm, vias 1 -> 0
- net Net-(JF31-Pad1): track 109.7 -> 0.00 mm, vias 1 -> 0
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Other:
- outline, holes or cut-outs redrawn
- board text added: "Zip-tie Battery Here"

Commit message: Laid out the middle PCB.
Parts:
- moved D13 42.5 mm to (72.8, 107.9)
- moved D14 42.5 mm to (72.8, 109.4)
- moved D19 25.4 mm to (99.0, 129.5), turned to 270 degrees
- moved D18 23.3 mm to (100.5, 129.5), turned to 270 degrees
- moved D28 23.1 mm to (193.6, 110.3), turned to 90 degrees
- moved D39 22.2 mm to (192.1, 110.3), turned to 90 degrees
- moved D40 21.3 mm to (190.6, 110.3), turned to 90 degrees
- moved D41 20.5 mm to (189.2, 110.3), turned to 90 degrees
- moved D49 20.1 mm to (130.2, 67.8)
- moved D42 19.9 mm to (187.7, 110.3), turned to 90 degrees
- moved D45 18.6 mm to (130.2, 66.3)
- moved D46 18.6 mm to (130.2, 64.8)
- moved D47 18.5 mm to (130.2, 63.3)
- moved D48 18.5 mm to (130.2, 61.8)
- moved D50 18.5 mm to (130.2, 60.3)
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Routing:
- net COL4: track 141.3 -> 499.8 mm, vias 1 -> 3
- net COL5: track 115.9 -> 397.4 mm, vias 1 -> 5
- net GND: track 206.8 -> 446.2 mm, vias 2 -> 11
- net COL2: track 191.7 -> 408.5 mm, vias 1 -> 4
- net COL3: track 177.1 -> 376.4 mm, vias 1 -> 6
- net ROWR4: track 37.2 -> 143.2 mm, vias 0 -> 1
- net COL0: track 97.2 -> 161.0 mm, vias 1 -> 2
- net ROWL4: track 80.2 -> 143.8 mm, vias 1 -> 3
- net COL1: track 139.2 -> 201.2 mm, vias 1 -> 2
- net ROWR3: track 0.00 -> 50.4 mm
- net Net-(D45-Pad2): track 0.00 -> 50.0 mm, vias 0 -> 1
- net Net-(D46-Pad2): track 0.00 -> 48.1 mm, vias 0 -> 1
- net Net-(D35-Pad2): track 0.00 -> 47.5 mm, vias 0 -> 1
- net Net-(D31-Pad2): track 0.00 -> 46.1 mm, vias 0 -> 1
- net ROWL3: track 51.3 -> 97.4 mm, vias 1 -> 3
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- added copper zone on B.Cu, net GND
- added copper zone on F.Cu, net GND
Other:
- outline, holes or cut-outs redrawn

Commit message: Added connector holes for the switch panels.
Parts:
- moved D13 2.44 mm to (74.8, 106.5)
- moved D14 2.44 mm to (74.8, 108.0)
Routing:
- net COL0: track 161.0 -> 157.8 mm
- net COL1: track 201.2 -> 198.0 mm
- net Net-(JM45-Pad1): track 77.3 -> 74.3 mm
- net Net-(JM45-Pad2): track 94.3 -> 91.8 mm
- net Net-(D15-Pad2): track 45.3 -> 47.5 mm
- net Net-(D14-Pad2): track 33.6 -> 35.1 mm
- net Net-(D13-Pad2): track 13.2 -> 14.6 mm
- net COL3: track 376.4 -> 375.2 mm
- net Net-(D1-Pad2): track 35.6 -> 36.6 mm
- net Net-(D3-Pad2): track 40.6 -> 40.1 mm
Other:
- outline, holes or cut-outs redrawn

Commit message: Laid out the top PCB.
Routing:
- net DR-TOP: track 0.00 -> 53.3 mm
- net GND-TOP: track 51.1 -> 29.3 mm
- net SCL-TOP: track 42.8 -> 27.6 mm
- net Net-(JM43-Pad2): track 27.5 -> 41.1 mm, vias 1 -> 0
- net Net-(JM45-Pad2): track 91.8 -> 100.6 mm, vias 2 -> 1
- net Net-(JM45-Pad1): track 74.3 -> 79.2 mm
- net Net-(JM45-Pad3): track 14.8 -> 10.9 mm
- net L3GND: track 7.62 -> 5.08 mm
- net Net-(JM45-Pad4): track 33.8 -> 35.3 mm
- net Net-(JM43-Pad4): track 29.2 -> 27.9 mm
- net SDA-TOP: track 25.1 -> 26.3 mm
- net VCC-TOP: track 19.7 -> 20.9 mm
- net Net-(JM5-Pad3): track 14.5 -> 13.6 mm
- net Net-(JM43-Pad3): track 14.2 -> 13.4 mm
- net Net-(JM43-Pad1): track 18.0 -> 17.5 mm
- added copper zone on F.Cu, net L1GND
