File: ThumbsUp.kicad_pcb (KiCad board)
At the start: 2 copper layers, 282 x 464.4 mm, 159 parts, among them J19 52559-1233, J32 Battery, SW2 SW_DIP_x01, U1 nice_nano

Commit message: Laid out the bottom PCB.
Routing:
- net Net-(JF33-Pad3): track 16.4 -> 242.8 mm, vias 0 -> 1
- net Net-(JF33-Pad4): track 16.5 -> 237.7 mm, vias 0 -> 1
- net Net-(JF33-Pad2): track 16.3 -> 189.1 mm, vias 0 -> 1
- net Net-(JF33-Pad1): track 16.1 -> 188.5 mm, vias 0 -> 1
- net Net-(JF20-Pad2): track 0.00 -> 168.3 mm, vias 0 -> 1
- net Net-(JF20-Pad1): track 0.00 -> 167.9 mm, vias 0 -> 1
- net Net-(JF23-Pad1): track 6.39 -> 140.8 mm, vias 0 -> 1
- net Net-(JF20-Pad3): track 0.00 -> 130.1 mm, vias 0 -> 1
- net Net-(JF20-Pad4): track 0.00 -> 107.9 mm, vias 0 -> 1
- net Net-(JF28-Pad1): track 0.00 -> 107.0 mm, vias 0 -> 1
- net Net-(JF23-Pad2): track 6.53 -> 107.0 mm, vias 0 -> 1
- net Net-(JF31-Pad1): track 0.00 -> 95.7 mm, vias 0 -> 1
- net Net-(JF3-Pad1): track 0.00 -> 95.2 mm, vias 0 -> 1
- net Net-(JF29-Pad1): track 0.00 -> 93.6 mm, vias 0 -> 1
- net Net-(JF30-Pad1): track 0.00 -> 93.2 mm, vias 0 -> 1
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
Commit message: Added silkscreens.
Parts:
- added G***: LOGO, Silkscreens:Crowfeet, B.Cu at (144.6, 281.3)
- added G***: LOGO, Silkscreens:Crowfeet, F.Cu at (142.6, 281.6)
- added G***: LOGO, Silkscreens:Crowfeet, F.Cu at (142.1, 90.9)
- added G***: LOGO, Silkscreens:Crowfeet, F.Cu at (142.5, -118.4)
