File: ThumbsUp_SwitchPlates.kicad_pcb (KiCad board)
At the start: 2 copper layers, 278.8 x 382.3 mm, 32 parts

Commit message: Added silkscreens.
Parts:
- added G***: LOGO, Silkscreens:Crowfeet, B.Cu at (144.0, 15.2)
- added G***: LOGO, Silkscreens:Crowfeet, B.Cu at (232.1, 236.7)
- added G***: LOGO, Silkscreens:Crowfeet, F.Cu at (229.7, 237.3)
- added G***: LOGO, Silkscreens:Crowfeet, F.Cu at (142.1, 15.1)

Commit message: Added solder mask areas to trim the silkscreen outside of the pcb.
Parts:
- moved G*** 8.37 mm to (233.7, 230.0)
- moved G*** 7.57 mm to (235.3, 229.8)
Changed lines of the file:
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@@
     (36 B.SilkS user)
     (37 F.SilkS user)
-    (38 B.Mask user hide)
-    (39 F.Mask user)
+    (38 B.Mask user)
+    (39 F.Mask user hide)
     (40 Dwgs.User user hide)
     (41 Cmts.User user)
@@
   )
   (module Silkscreens:Crowfeet (layer B.Cu)
-    (at 232.145 236.7124 180)
+    (at 235.295 229.8324 180)
     (fp_text reference G*** (at 0 0) (layer B.SilkS) hide
       (effects (font (size 1.524 1.524) (thickness 0.3)) (justify mirror))
@@
   )
   (module Silkscreens:Crowfeet (layer F.Cu)
-    (at 229.655 237.2924)
+    (at 233.705 229.9624)
     (fp_text reference G*** (at 0 0) (layer F.SilkS) hide
       (effects (font (size 1.524 1.524) (thickness 0.3)))
@@
   (gr_line (start 209.758126 -86.081962) (end 176.347118 -72.577216) (layer Edge.Cuts) (width 0.05))
   (gr_line (start 220.409281 -72.265924) (end 176.161819 -38.965742) (layer Edge.Cuts) (width 0.05))
+  (zone (net 0) (net_name "") (layer F.Mask) (hatch edge 0.508)
+    (connect_pads (clearance 0.508))
+    (min_thickness 0.254)
+    (fill yes (arc_segments 32) (thermal_gap 0.508) (thermal_bridge_width 0.508))
+    (polygon
+      (pts
+        (xy 255.145 121.8824) (xy 255.095 189.8924) (xy 258.565 190.5924) (xy 285.275 257.8024) (xy 283.365 261.9724)
+        (xy 270.535 266.1324) (xy 267.755 273.2424) (xy 212.765 294.4324) (xy 181.545 214.8124) (xy 182.585 212.2124)
+        (xy 203.225 203.5424) (xy 208.265 207.0124) (xy 251.625 189.1624) (xy 251.625 122.3224) (xy 44.395 123.8824)
+        (xy 46.305 340.1924) (xy 425.395 337.4124) (xy 422.445 123.5924)
+      )
+    )
+  )
+  (zone (net 0) (net_name "") (layer F.Mask) (hatch edge 0.508)
+    (connect_pads (clearance 0.508))
+    (min_thickness 0.254)
+    (fill yes (arc_segments 32) (thermal_gap 0.508) (thermal_bridge_width 0.508))
+    (polygon
+      (pts
+        (xy 247.775 123.4224) (xy 248.295 188.4624) (xy 259.045 188.9824) (xy 257.315 124.9824) (xy 258.185 124.6324)
+        (xy 257.665 123.4224)
+      )
+    )
+  )
+  (zone (net 0) (net_name "") (layer B.Mask) (hatch edge 0.508)
+    (connect_pads (clearance 0.508))
+    (min_thickness 0.254)
+    (fill yes (arc_segments 32) (thermal_gap 0.508) (thermal_bridge_width 0.508))
+    (polygon
+      (pts
+        (xy 257.835 189.5024) (xy 258.525 124.6624) (xy 422.965 124.1424) (xy 421.405 338.2424) (xy 45.125 336.6824)
+        (xy 47.725 123.8624) (xy 254.655 124.9024) (xy 255.185 189.0824) (xy 222.745 201.9124) (xy 219.105 201.7424)
+        (xy 208.525 206.0824) (xy 201.235 203.6524) (xy 180.425 211.9824) (xy 214.595 294.6024) (xy 269.395 272.4024)
+        (xy 270.785 266.5024) (xy 283.795 261.4724) (xy 285.705 257.3124)
+      )
+    )
+  )
+  (zone (net 0) (net_name "") (layer B.Mask) (hatch edge 0.508)
+    (connect_pads (clearance 0.508))
+    (min_thickness 0.254)
+    (fill yes (arc_segments 32) (thermal_gap 0.508) (thermal_bridge_width 0.508))
+    (polygon
+      (pts
+        (xy 251.355 122.8324) (xy 251.355 187.3624) (xy 263.325 192.3924) (xy 260.725 122.3124)
+      )
+    )
+  )
 )
